File: PCBs/power_module/power_module.kicad_sch (KiCad schematic)
At the start: 5 parts, among them K1 SANYOU_SRD_Form_C, K2 SANYOU_SRD_Form_C, K3 SANYOU_SRD_Form_C, K4 SANYOU_SRD_Form_C, K5 SANYOU_SRD_Form_C

Commit message: updated power_module pcb
updated power_module pcb
Parts:
- added C1, C2, C24, C25, C3, C43, C45, C46, C7: 3.3uF, Capacitors_SMD:C_0603_HandSoldering, symbol pspice:CAP
- added C10, C29, C50: 0.022uF, Capacitors_SMD:C_0603_HandSoldering, symbol Device:C
- added C11, C16, C17, C26, C27, C44, C47, C48, C8: OPT, Capacitors_SMD:C_0603_HandSoldering, symbol Device:C
- added C12, C20, C23, C31, C33, C40, C52, C54, C61: 0.01uF, Capacitors_SMD:C_0603_HandSoldering, symbol Device:C
- added C13, C34, C55: 47pF, Capacitors_SMD:C_0603_HandSoldering, symbol Device:C
- added C14, C41, C62: 0.1uF, Capacitors_SMD:C_0603_HandSoldering, symbol Device:C
- added C15, C39, C60: 1uF, Capacitors_SMD:C_0603_HandSoldering, symbol Device:C
- added C18, C42, C63: 4.7uF, Capacitors_SMD:C_0603_HandSoldering, symbol Device:C
- added C19, C36, C57: 1000pF, Capacitors_SMD:C_0603_HandSoldering, symbol Device:C
- added C21, C35, C56: 100pF, Capacitors_SMD:C_0603_HandSoldering, symbol Device:C
- added C22, C37, C38, C4, C58, C59: 0.22uF, Capacitors_SMD:C_0603_HandSoldering, symbol Device:C
- added C28, C30, C32, C49, C5, C51, C53, C6, C9: 22uF, Capacitors_SMD:C_0603_HandSoldering, symbol pspice:CAP
- added CIN1, CIN2, CIN3, CIN4, CIN5, CIN6: 22uF, Capacitors_SMD:CP_Elec_8x6.7, symbol Device:CP
- added COUT1, COUT2, COUT3, COUT4, COUT5, COUT6: 330uF, Capacitors_SMD:CP_Elec_8x10.5, symbol Device:CP
- added D1, D11, D17: 4.7V, Diodes_SMD:D_SOD-323_HandSoldering, symbol Device:D_Zener
- added D10, D12, D16, D18, D4, D7: 1N819HW, Diodes_SMD:D_SOD-123, symbol Device:D_Zener
- added D13, D2, D3: 36V, Diodes_SMD:D_SOT-23_ANK, symbol Device:D_Zener
- added D14, D15, D5, D6, D8, D9: B320A, Diodes_SMD:D_SMA_Handsoldering, symbol Device:D_Zener
- added H1, H10, H11, H12, H2, H3, H4, H5, H6, H7, H8, H9: MountingHole, Mounting_Holes:MountingHole_4mm, symbol Mechanical:MountingHole
- added J1, J2, J3, J4, J5, J6: Screw_Terminal_01x02, Connectors_JST:JST_VH_B2P-VH_2x3.96mm_Vertical, symbol Connector:Screw_Terminal_01x02
- added L1, L2, L3: 4.7uH, Inductors:Inductor_Wurth_MAPI-4020, symbol pspice:INDUCTOR
- added PLL_IN1, PLL_IN2, PLL_IN3: TestPoint, Measurement_Points:Measurement_Point_Square-SMD-Pad_Small, symbol Connector:TestPoint
- added Q1, Q10, Q11, Q12, Q2, Q3, Q4, Q5, Q6, Q7, Q8, Q9: IPD100N04S402ATMA1, TO_SOT_Packages_SMD:TO-252-2, symbol Transistor_FET:IPD100N04S402ATMA1
- added R1, R17, R20, R30, R32, R36, R48, R50, R54: 10K, Resistors_SMD:R_0603_HandSoldering, symbol Device:R
- added R10, R22, R39, R40, R7, R9: 1K24, Resistors_SMD:R_0603_HandSoldering, symbol Device:R
- added R11, R31, R49: 100K, Resistors_SMD:R_0603_HandSoldering, symbol Device:R
- added R12, R26, R44: 113K, Resistors_SMD:R_0603_HandSoldering, symbol Device:R
- added R13, R27, R45: 8.06K, Resistors_SMD:R_0603_HandSoldering, symbol Device:R
- added R14, R16, R28, R29, R46, R47: OPT, Resistors_SMD:R_0603_HandSoldering, symbol Device:R
- added R15, R33, R51: 220k, Resistors_SMD:R_0603_HandSoldering, symbol Device:R
- added R18, R19, R3, R37, R38, R6: 0.018R, Resistors_SMD:R_2512_HandSoldering, symbol Device:R
- added R2, R23, R24, R4, R41, R42: 0R, Resistors_SMD:R_0603_HandSoldering, symbol Device:R
- added R21, R34, R52: DNF, Resistors_SMD:R_0603_HandSoldering, symbol Device:R
- added R25, R35, R43, R5, R53, R8: 10R, Resistors_SMD:R_0603_HandSoldering, symbol Device:R
- added U1, U2, U3: LTC3780EGPBF, LTC3780EGPBF:SOP65P780X200-24N, symbol LTC3780EGPBF:LTC3780EGPBF
Connections:
- net GND: now also C1.2, C10.2, C12.2, C13.2, C14.2, C15.1, C17.2, C18.2, C19.2, C2.2, C21.2, C23.2, C24.2, C25.2, C27.2, C28.2, C29.2, C3.2, C30.2, C31.2, C32.2, C34.2, C35.2, C36.2, C39.1, C40.2, C41.2, C42.2, C43.2, C45.2, C46.2, C48.2, C49.2, C5.2, C50.2, C51.2, C52.2, C53.2, C55.2, C56.2, C57.2, C6.2, C60.1, C61.2, C62.2, C63.2, C7.2, C9.2, CIN1.2, CIN2.2, CIN3.2, CIN4.2, CIN5.2, CIN6.2, COUT1.2, COUT2.2, COUT3.2, COUT4.2, COUT5.2, COUT6.2, D1.2 (A), D11.2 (A), D13.2 (A), D17.2 (A), D2.2 (A), D3.2 (A), J1.1 (Pin_1), J2.1 (Pin_1), J3.1 (Pin_1), J4.1 (Pin_1), J5.1 (Pin_1), J6.1 (Pin_1), R10.2, R13.2, R17.2, R18.2, R19.2, R20.2, R22.2, R27.2, R3.2, R30.2, R32.2, R37.2, R38.2, R40.2, R45.2, R48.2, R50.2, R6.2, U1.17 (PGND), U1.7 (SGND), U2.17 (PGND), U2.7 (SGND), U3.17 (PGND), U3.7 (SGND)
- new net: R36.2, U1.1 (PGOOD)
- new net: PLL_IN2.1, U1.11 (PLLIN)
- new net: C40.1, R34.2, U1.12 (STBYMD)
- new net: C37.1, D10.1 (K), U1.13 (BOOST2)
- new net: C29.1, U1.2 (SS)
- new net: C39.2, U1.20 (EXTVCC)
- new net: C41.1, R35.2, U1.21 (VIN)
- new net: C38.1, D12.1 (K), U1.24 (BOOST1)
- new net: C34.1, R31.1, U1.5 (ITH)
- new net: D11.1 (K), R33.2, U1.8 (RUN)
- new net: C36.1, U1.9 (FCB)
- new net: C14.1, R5.2, U2.21 (VIN)
- new net: R1.2, U2.1 (PGOOD)
- new net: C23.1, R21.2, U2.12 (STBYMD)
- new net: PLL_IN1.1, U2.11 (PLLIN)
- new net: C10.1, U2.2 (SS)
- new net: C13.1, R11.1, U2.5 (ITH)
- new net: C12.1, R11.2
- new net: C19.1, U2.9 (FCB)
- new net: C16.2, R12.1, R8.2
- new net: C16.1, R16.1
- new net: C17.1, R14.1
- new net: D6.2 (A), Q4.3, Q5.3, R18.1, R19.1, R9.2
- new net: D1.1 (K), R15.2, U2.8 (RUN)
- new net: C20.2, R17.1
- new net: C15.2, U2.20 (EXTVCC)
- new net: C4.1, D4.1 (K), U2.24 (BOOST1)
- new net: C22.1, D7.1 (K), U2.13 (BOOST2)
- new net: C11.1, R2.2, R9.1
- new net: C11.2, R10.1, R4.2
- new net: C26.2, R25.2, R26.1
- new net: C27.1, R28.1
- new net: C47.2, R43.2, R44.1
- new net: C55.1, R49.1, U3.5 (ITH)
- new net: C8.1, R23.2, R7.1
- new net: D17.1 (K), R51.2, U3.8 (RUN)
- new net: C61.1, R52.2, U3.12 (STBYMD)
- new net: C8.2, R22.1, R24.2
- new net: C44.2, R40.1, R42.2
- new net: C44.1, R39.1, R41.2
- new net: D14.2 (A), Q10.3, Q12.3, R37.1, R38.1, R39.2
- new net: C50.1, U3.2 (SS)
- new net: C31.1, R31.2
- new net: D8.2 (A), Q6.3, Q8.3, R3.1, R6.1, R7.2
- new net: C59.1, D18.1 (K), U3.24 (BOOST1)
- new net: C47.1, R47.1
- new net: C62.1, R53.2, U3.21 (VIN)
- new net: C58.1, D16.1 (K), U3.13 (BOOST2)
- new net: C54.2, R48.1
- new net: C33.2, R30.1
- new net: C26.1, R29.1
- new net: C60.2, U3.20 (EXTVCC)
- new net: C52.1, R49.2
- new net: C57.1, U3.9 (FCB)
- new net: R54.2, U3.1 (PGOOD)
- new net: C48.1, R46.1
- new net: PLL_IN3.1, U3.11 (PLLIN)
- new net +6V: C18.1, C42.1, C63.1, D10.2 (A), D12.2 (A), D16.2 (A), D18.2 (A), D4.2 (A), D7.2 (A), R1.1, R36.1, R54.1, U1.19 (INTVCC), U2.19 (INTVCC), U3.19 (INTVCC)
- new net +VSW: C1.1, C2.1, C24.1, C25.1, C3.1, C43.1, C45.1, C46.1, C7.1, CIN1.1, CIN2.1, CIN3.1, CIN4.1, CIN5.1, CIN6.1, D13.1 (K), D2.1 (K), D3.1 (K), J1.2 (Pin_2), J3.2 (Pin_2), J5.2 (Pin_2), Q1.2, Q3.2, Q9.2, R15.1, R21.1, R33.1, R34.1, R35.1, R5.1, R51.1, R52.1, R53.1
- new net BG1: Q12.1, Q4.1, Q8.1, U1.18 (BG1), U2.18 (BG1), U3.18 (BG1)
- new net BG2: Q10.1, Q5.1, Q6.1, U1.16 (BG2), U2.16 (BG2), U3.16 (BG2)
- new net PLLFILTR: C20.1, C21.1, C33.1, C35.1, C54.1, C56.1, R20.1, R32.1, R50.1, U1.10 (PLLFLTR), U2.10 (PLLFLTR), U3.10 (PLLFLTR)
- new net SENSE+: R2.1, R23.1, R41.1, U1.3 (SENSE+), U2.3 (SENSE+), U3.3 (SENSE+)
- new net SENSE-: R24.1, R4.1, R42.1, U1.4 (SENSE-), U2.4 (SENSE-), U3.4 (SENSE-)
- new net SW1: C38.2, C4.2, C59.2, D15.2 (A), D5.2 (A), D9.2 (A), L1.2, L2.2, L3.2, Q11.3, Q12.2, Q2.3, Q4.2, Q7.3, Q8.2, U1.22 (SW1), U2.22 (SW1), U3.22 (SW1)
- new net SW2: C22.2, C37.2, C58.2, D14.1 (K), D6.1 (K), D8.1 (K), L1.1, L2.1, L3.1, Q1.3, Q10.2, Q3.3, Q5.2, Q6.2, Q9.3, U1.15 (SW2), U2.15 (SW2), U3.15 (SW2)
- new net TG1: Q11.1, Q2.1, Q7.1, U1.23 (TG1), U2.23 (TG1), U3.23 (TG1)
- new net TG2: Q1.1, Q3.1, Q9.1, U1.14 (TG2), U2.14 (TG2), U3.14 (TG2)
- new net VCC: C28.1, C30.1, C32.1, C49.1, C5.1, C51.1, C53.1, C6.1, C9.1, COUT1.1, COUT2.1, COUT3.1, COUT4.1, COUT5.1, COUT6.1, D15.1 (K), D5.1 (K), D9.1 (K), J2.2 (Pin_2), J4.2 (Pin_2), J6.2 (Pin_2), Q11.2, Q2.2, Q7.2, R25.1, R43.1, R8.1
- new net VSENSE: R12.2, R13.1, R14.2, R16.2, R26.2, R27.1, R28.2, R29.2, R44.2, R45.1, R46.2, R47.2, U1.6 (VOSENSE), U2.6 (VOSENSE), U3.6 (VOSENSE)
Other:
- company: (none) -> UMD Loop
- title: (none) -> Power PCB
