File: PCBs/REALFLURO/REALFLURO.kicad_pcb (KiCad board)
At the start: 2 copper layers, 3 parts, among them J1 Conn_02x07_Odd_Even, J2 Conn_02x08_Odd_Even, J3 Conn_02x08_Odd_Even

Commit message: v1 power pcb w/ led level shifter
Parts:
- added D1: LED, LED_THT:LED_D3.0mm_Horizontal_O1.27mm_Z2.0mm_Clear, F.Cu at (150.3, 68.3)
- added R1: 100, Resistor_SMD:R_0201_0603Metric, F.Cu at (144.5, 71.5)
- added U1: OPT101P, OPT101P:DIP762W46P254L952H419Q8, F.Cu at (137.3, 65.6)
Routing:
- net GND: track 0.00 -> 30.5 mm
- net /59: track 0.00 -> 9.91 mm
- net Net-(D1-A): track 0.00 -> 4.37 mm
- net +5V: track 0.00 -> 3.98 mm
Other:
- board outline added: 32.2 x 34.2 mm
