File: PCBs/3-DOF/3-DOF.kicad_sch (KiCad schematic)
At the start: 43 parts, among them J1 Conn_02x07_Odd_Even, J10 Conn_01x06, J12 Conn_01x04, J13 Conn_01x03, J14 Conn_01x04, J15 Conn_01x04, J16 Conn_01x04, J17 Conn_01x04, J18 Conn_01x04, J2 Conn_02x08_Odd_Even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

Commit message: minor fixes
Connections:
- net 26: no longer J14.4 (Pin_4)
- net 27: no longer J15.4 (Pin_4)
- net 28: no longer J16.4 (Pin_4)
- no-connect marks 4 -> 7
Other:
- moved on the sheet: C15, C16, J17, J18

Commit message: bug fixes
Parts:
- removed C12, C13, C14: 10u, Capacitor_SMD:C_0402_1005Metric_Pad0.74x0.62mm_HandSolder, symbol Device:C
- removed J13: Conn_01x03, Connector_JST:JST_XH_S3B-XH-A_1x03_P2.50mm_Horizontal, symbol Connector_Generic:Conn_01x03
- removed J14, J15, J16: Conn_01x04, Connector_JST:JST_XH_S4B-XH-A_1x04_P2.50mm_Horizontal, symbol Connector_Generic:Conn_01x04
- removed Q1: 2N7000, Package_TO_SOT_THT:TO-92_Inline, symbol Transistor_FET:2N7000
- removed R2: 100, Resistor_SMD:R_0402_1005Metric_Pad0.72x0.64mm_HandSolder, symbol Device:R_US
- added C17, C18: 470u, Capacitor_SMD:C_0402_1005Metric_Pad0.74x0.62mm_HandSolder, symbol Device:C
- added J9: Conn_01x02, symbol Connector_Generic:Conn_01x02
- J17: footprint Connector_JST:JST_XH_S4B-XH-A_1x04_P2.50mm_Horizontal -> Connector_JST:JST_GH_SM04B-GHS-TB_1x04-1MP_P1.25mm_Horizontal
- U2, U3: footprint Package_TO_SOT_THT:TO-220-15_P2.54x5.08mm_StaggerOdd_Lead4.58mm_Vertical -> footprints:l298n_with_heatsink
Connections:
- net +24V: now also C17.2, C18.2
- net +5V: now also J17.2 (Pin_2), J18.2 (Pin_2); no longer J17.1 (Pin_1), J18.1 (Pin_1)
- net GND: now also J17.1 (Pin_1), J18.1 (Pin_1), U2.1 (SENSE_A), U2.15 (SENSE_B), U3.1 (SENSE_A), U3.15 (SENSE_B), C17.1, C18.1, J9.2 (Pin_2); no longer J17.2 (Pin_2), J18.2 (Pin_2)
- no-connect marks 7 -> 0
Other:
- moved on the sheet: C15, J18
