File: PCBs/3-DOF/3-DOF.kicad_sch (KiCad schematic)
At the start: 78 parts, among them J1 Conn_02x07_Odd_Even, J11 Conn_01x06, J12 Conn_01x04, J13 Conn_01x06, J14 Conn_01x06, J15 Conn_01x06, J17 Conn_01x04, J18 Conn_01x04, J2 Conn_02x08_Odd_Even, J3 Conn_02x08_Odd_Even, J5 Conn_01x02, J9 Conn_01x02, Q1 S8050, Q2 S8550, Q3 S8050, Q4 S8550, Q5 S8550, U1 MAX485E, U2 LM7805_TO220, U3 AMS1117CD-3.3, U4 L298N, U5 L298N

Commit message: 80% routed
Parts:
- removed C4, C9: 10u, Capacitor_SMD:C_0805_2012Metric_Pad1.18x1.45mm_HandSolder, symbol Device:C
- removed C8: 22u, Capacitor_SMD:C_0805_2012Metric_Pad1.18x1.45mm_HandSolder, symbol Device:C
- removed Q5: S8550, Package_TO_SOT_THT:TO-92_Inline, symbol Transistor_BJT:S8550
- removed R13: 220, Resistor_SMD:R_0402_1005Metric_Pad0.72x0.64mm_HandSolder, symbol Device:R
- removed R14: 330, Resistor_SMD:R_0402_1005Metric_Pad0.72x0.64mm_HandSolder, symbol Device:R
- removed R15: 680, Resistor_SMD:R_0402_1005Metric_Pad0.72x0.64mm_HandSolder, symbol Device:R
- removed U3: AMS1117CD-3.3, Package_TO_SOT_SMD:TO-252-3_TabPin2, symbol Regulator_Linear:AMS1117CD-3.3
- added CLD1: 10u, Capacitor_SMD:C_0805_2012Metric_Pad1.18x1.45mm_HandSolder, symbol Device:C
- added CVregA3, CVregA4: 100n, Capacitor_SMD:C_0805_2012Metric_Pad1.18x1.45mm_HandSolder, symbol Device:C
- added LaserDiodeT1: S8550, Package_TO_SOT_THT:TO-92_Inline, symbol Transistor_BJT:S8550
- added Q6: LaserDiodeT, Package_TO_SOT_THT:TO-92_Inline, symbol Transistor_BJT:S8050
- added RLD1: 220, Resistor_SMD:R_0402_1005Metric_Pad0.72x0.64mm_HandSolder, symbol Device:R
- added RLD2: 330, Resistor_SMD:R_0402_1005Metric_Pad0.72x0.64mm_HandSolder, symbol Device:R
- added RLD3: 680, Resistor_SMD:R_0402_1005Metric_Pad0.72x0.64mm_HandSolder, symbol Device:R
- added U3: LM7805_TO220, Package_TO_SOT_SMD:SOT-23_Handsoldering, symbol Regulator_Linear:LM7805_TO220
- CVregA1: renamed from C1; value .33u -> 100n
- CVregA2: renamed from C2; value .1u -> 100n
- J11, J13: value Conn_01x06 -> HBB
- J12: value Conn_01x04 -> RS485
- J14, J15: value Conn_01x06 -> HBA
- J17: value Conn_01x04 -> Servo1
- J5: value Conn_01x02 -> 24Vin; footprint Connector_JST:JST_GH_SM02B-GHS-TB_1x02-1MP_P1.25mm_Horizontal -> Connector_Molex:Molex_Micro-Fit_3.0_43650-0210_1x02-1MP_P3.00mm_Horizontal
- J9: value Conn_01x02 -> Laser Diode
- Q1: value S8050 -> QServoA
- renumbered C19 to CHBA1, C24 to CHBA2, C25 to CHBA3, C20 to CHBA4, C23 to CHBA5, C14 to CHBB1, C21 to CHBB2, C22 to CHBB3, C15 to CHBB4, C16 to CHBB5, C6 to CRS1, C5 to CRS2, C7 to CRS3, C13 to CServoA1, C12 to CServoB1, C3 to CVin1, D9 to DHBA1, D10 to DHBA2, D11 to DHBA3, D12 to DHBA4, D13 to DHBA5, D14 to DHBA6, D15 to DHBA7, D16 to DHBA8, D5 to DHBB1, D1 to DHBB2, D6 to DHBB3, D2 to DHBB4, D3 to DHBB5, D7 to DHBB6, D4 to DHBB7, D8 to DHBB8, J18 to JServoB1, Q2 to QServoA1, Q3 to QServoB1, Q4 to QServoB2, R1 to RRS1, R3 to RRS2, R4 to RRS3, R6 to RRS4, R5 to RRS5, R7 to RRS6, R10 to RServoA1, R11 to RServoA2, R12 to RServoA3, R2 to RServoB1, R8 to RServoB2, R9 to RServoB3, U5 to UHBA1, U4 to UHBB1
Connections:
- net +3.3V: now also CHBA4.1, CHBA5.1, CHBB2.1, CHBB3.1, CRS2.2, J11.5 (Pin_5), J13.5 (Pin_5), J14.5 (Pin_5), J15.5 (Pin_5), RRS1.1, RRS2.1, RRS3.1, RRS5.1, U1.8 (VCC), CVregA3.1, U3.2 (Vout); no longer CRS3.1, J12.1 (Pin_1)
- net +5V: now also CRS3.1, J12.1 (Pin_1), CLD1.2, CVregA4.1, LaserDiodeT1.1 (E), RLD2.2, U3.3 (Vin); no longer CHBA4.1, CHBA5.1, CHBB2.1, CHBB3.1, CRS2.2, J11.5 (Pin_5), J13.5 (Pin_5), J14.5 (Pin_5), J15.5 (Pin_5), RRS1.1, RRS2.1, RRS3.1, RRS5.1, U1.8 (VCC)
- net 56: now also RLD1.1
- net GND: now also CLD1.1, CVregA3.2, CVregA4.2, Q6.1 (E), U3.1 (GND)
- net at J9.1 (Pin_1): now also LaserDiodeT1.3 (C)
- new net: LaserDiodeT1.2 (B), RLD2.1, RLD3.2
- new net: Q6.2 (B), RLD1.2
- new net: Q6.3 (C), RLD3.1
