File: PCBs/3-DOF/3-DOF.kicad_pcb (KiCad board)
At the start: 2 copper layers, 78 parts, among them J1 Conn_02x07_Odd_Even, J11 Conn_01x06, J12 Conn_01x04, J13 Conn_01x06, J14 Conn_01x06, J15 Conn_01x06, J17 Conn_01x04, J18 Conn_01x04, J2 Conn_02x08_Odd_Even, J3 Conn_02x08_Odd_Even, J5 Conn_01x02, J9 Conn_01x02, Q1 S8050, Q2 S8550, Q3 S8050, Q4 S8550, Q5 S8550, U1 MAX485E, U2 LM7805_TO220, U3 AMS1117CD-3.3, U4 L298N, U5 L298N

Commit message: 80% routed
Parts:
- removed C8: 22u, Capacitor_SMD:C_0805_2012Metric_Pad1.18x1.45mm_HandSolder
- removed C9: 10u, Capacitor_SMD:C_0805_2012Metric_Pad1.18x1.45mm_HandSolder
- removed R15: 680, Resistor_SMD:R_0402_1005Metric_Pad0.72x0.64mm_HandSolder
- added CLD1: 10u, Capacitor_SMD:C_0805_2012Metric_Pad1.18x1.45mm_HandSolder, F.Cu at (162.9, 79.3)
- added CVregA3: 100n, Capacitor_SMD:C_0805_2012Metric_Pad1.18x1.45mm_HandSolder, F.Cu at (162.9, 81.6)
- added CVregA4: 100n, Capacitor_SMD:C_0805_2012Metric_Pad1.18x1.45mm_HandSolder, F.Cu at (158.2, 53.3)
- added LaserDiodeT1: S8550, Package_TO_SOT_THT:TO-92_Inline, F.Cu at (167.5, 81.3)
- added Q6: LaserDiodeT, Package_TO_SOT_THT:TO-92_Inline, F.Cu at (174.8, 81.9)
- added RLD1: 220, Resistor_SMD:R_0402_1005Metric_Pad0.72x0.64mm_HandSolder, F.Cu at (155.0, 80.5)
- added RLD2: 330, Resistor_SMD:R_0402_1005Metric_Pad0.72x0.64mm_HandSolder, F.Cu at (131.7, 82.3)
- added RLD3: 680, Resistor_SMD:R_0402_1005Metric_Pad0.72x0.64mm_HandSolder, F.Cu at (144.5, 82.0)
- CVregA1: renamed from C1; value .33u -> 100n
- CVregA2: renamed from C2; value .1u -> 100n
- J11, J13: value Conn_01x06 -> HBB
- J12: value Conn_01x04 -> RS485
- J14, J15: value Conn_01x06 -> HBA
- J17: value Conn_01x04 -> Servo1
- J5: value Conn_01x02 -> 24Vin; footprint Connector_JST:JST_GH_SM02B-GHS-TB_1x02-1MP_P1.25mm_Horizontal -> Connector_Molex:Molex_Micro-Fit_3.0_43650-0210_1x02-1MP_P3.00mm_Horizontal
- J9: value Conn_01x02 -> Laser Diode
- Q1: value S8050 -> QServoA
- U3: value AMS1117CD-3.3 -> LM7805_TO220; footprint Package_TO_SOT_SMD:TO-252-3_TabPin2 -> Package_TO_SOT_SMD:SOT-23_Handsoldering
- moved RServoA2 126.3 mm to (118.1, 50.5)
- moved RServoA1 123.5 mm to (120.8, 48.9), turned to 90 degrees
- moved RRS6 121.0 mm to (115.8, 76.5), turned to 90 degrees
- moved RRS5 120.2 mm to (116.6, 74.6), turned to 180 degrees
- moved RRS4 119.4 mm to (117.4, 76.4), turned to -90 degrees
- moved RServoB3 118.7 mm to (121.2, 79.0), turned to 90 degrees
- moved RServoA3 118.4 mm to (126.5, 51.7), turned to 180 degrees
- moved H2 116.8 mm to (103.7, 89.1)
- moved RServoB2 115.6 mm to (121.0, 86.7), turned to -90 degrees
- moved RServoB1 113.7 mm to (119.7, 79.0), turned to 90 degrees
- moved RRS1 112.7 mm to (122.0, 62.8), turned to 90 degrees
- moved QServoB1 112.0 mm to (121.2, 73.4), turned to -90 degrees
- moved H1 109.8 mm to (101.6, 46.5)
- moved CServoA1 107.7 mm to (118.0, 54.1), turned to 90 degrees
- moved Q1 107.2 mm to (124.5, 54.4), turned to 180 degrees
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- renumbered C19 to CHBA1, C24 to CHBA2, C25 to CHBA3, C20 to CHBA4, C23 to CHBA5, C14 to CHBB1, C21 to CHBB2, C22 to CHBB3, C15 to CHBB4, C16 to CHBB5, C6 to CRS1, C5 to CRS2, C7 to CRS3, C13 to CServoA1, C12 to CServoB1, C3 to CVin1, C4 to CVregB1, D9 to DHBA1, D10 to DHBA2, D11 to DHBA3, D12 to DHBA4, D13 to DHBA5, D14 to DHBA6, D15 to DHBA7, D16 to DHBA8, D5 to DHBB1, D1 to DHBB2, D6 to DHBB3, D2 to DHBB4, D3 to DHBB5, D7 to DHBB6, D4 to DHBB7, D8 to DHBB8, J18 to JServoB1, Q2 to QServoA1, Q3 to QServoB1, Q4 to QServoB2, R1 to RRS1, R3 to RRS2, R4 to RRS3, R6 to RRS4, R5 to RRS5, R7 to RRS6, R10 to RServoA1, R11 to RServoA2, R12 to RServoA3, R2 to RServoB1, R8 to RServoB2, R9 to RServoB3, U5 to UHBA1, U4 to UHBB1
Connections:
- CHBA4 pad 1: +5V -> +3.3V
- CHBA5 pad 1: +5V -> +3.3V
- CHBB2 pad 1: +5V -> +3.3V
- CHBB3 pad 1: +5V -> +3.3V
- CRS2 pad 2: +5V -> +3.3V
- CRS3 pad 1: +3.3V -> +5V
- J11 pad 5: +5V -> +3.3V
- J12 pad 1: +3.3V -> +5V
- J13 pad 5: +5V -> +3.3V
- J14 pad 5: +5V -> +3.3V
- J15 pad 5: +5V -> +3.3V
- RRS1 pad 1: +5V -> +3.3V
- RRS2 pad 1: +5V -> +3.3V
- RRS3 pad 1: +5V -> +3.3V
- RRS5 pad 1: +5V -> +3.3V
- U1 pad 8: +5V -> +3.3V
Routing:
- net +24V: track 0.00 -> 177.1 mm
- net +3.3V: track 0.00 -> 139.0 mm, vias 0 -> 14
- net GND: track 0.00 -> 101.9 mm, vias 0 -> 52
- net /55: track 0.00 -> 68.4 mm
- net Net-(DHBB1-A): track 0.00 -> 60.3 mm, vias 0 -> 1
- net /38: track 0.00 -> 53.6 mm
- net Net-(DHBA1-A): track 0.00 -> 52.0 mm, vias 0 -> 3
- net Net-(DHBB7-K): track 0.00 -> 47.1 mm, vias 0 -> 1
- net Net-(LaserDiodeT1-B): track 0.00 -> 44.6 mm, vias 0 -> 2
- net +5V: track 0.00 -> 43.5 mm, vias 0 -> 23
- net /37: track 0.00 -> 41.5 mm, vias 0 -> 2
- net /25: track 0.00 -> 40.5 mm, vias 0 -> 2
- net /11: track 0.00 -> 38.8 mm, vias 0 -> 1
- net Net-(DHBB5-K): track 0.00 -> 35.6 mm, vias 0 -> 1
- net /62: track 0.00 -> 34.7 mm, vias 0 -> 1
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- added copper zone on In2.Cu, net +5V
- added copper zone on In1.Cu, net GND
Other:
- board outline added: 97.1 x 53.8 mm
- copper layers 2 -> 4
- board text added: "${REFERENCE}"
