File: PCBs/3-DOF/3-DOF_PCB/3-DOF_PCB.kicad_pcb (KiCad board)
At the start: 4 copper layers, 97.1 x 53.8 mm, 83 parts, among them J1 Conn_02x07_Odd_Even, J11 HBB, J12 RS485, J13 HBB, J14 HBA, J15 HBA, J17 Servo1, J2 Conn_02x08_Odd_Even, J3 Conn_02x08_Odd_Even, J5 24Vin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

Commit message: init 2dof commit
Parts:
- moved H4 12.9 mm to (187.7, 84.7)
- moved H2 5.81 mm to (105.9, 83.7)
- turned DHBA8 to -90 degrees
Routing:
- net /26: track 38.2 -> 151.0 mm
- net GND: track 77.6 -> 124.2 mm, vias 36 -> 31
- net /56: track 35.5 -> 70.9 mm, vias 1 -> 0
- net +3.3V: track 189.3 -> 220.6 mm
- net Net-(DHBA1-A): track 57.9 -> 29.8 mm, vias 2 -> 1
- net /37: track 37.9 -> 58.1 mm, vias 1 -> 0
- net /30: track 33.2 -> 50.5 mm
- net Net-(Q1-B): track 7.61 -> 22.7 mm, vias 1 -> 0
- net /8: track 22.3 -> 34.5 mm, vias 1 -> 0
- net +5V: track 248.3 -> 257.1 mm
- net /62: track 47.3 -> 55.6 mm, vias 1 -> 0
- net /22: track 21.0 -> 13.8 mm, vias 1 -> 2
- net Net-(DHBB5-K): track 50.2 -> 57.3 mm, vias 2 -> 0
- net Net-(DHBA5-K): track 39.8 -> 44.9 mm, vias 3 -> 1
- net Net-(DHBB3-A): track 60.9 -> 65.6 mm, vias 3 -> 0
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Other:
- board size 97.1 x 53.8 mm -> 97 x 50.8 mm
