File: PCBs/2Dof/2Dof.kicad_pcb (KiCad board)
At the start: 2 copper layers, 53.1 x 46 mm, 50 parts, among them J1 Conn_02x07_Odd_Even, J12 RS485, J14 HBA, J17 Servo1, J2 Conn_02x08_Odd_Even, J3 Conn_02x08_Odd_Even, J5 24Vin, J9 Laser Diode, Q1 QServoA, Q6 LaserDiodeT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

Commit message: first review
Other:
- board text added: "In the box I made, the routings not great, a lot of places have vias where they dont need if the routing and placement was done better. An example of this is the resistor for the transciever (RRS4?) Is super far away from the transciever so it leads to you using vias where not needed you should have a 10uf at the 24V input header, also you should move it further from the hbridge since the heatsin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"
Changed lines of the file:
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@@
 		(layer "Edge.Cuts")
+	)
+	(gr_rect
+		(start 118.25 49.13)
+		(end 145.3 64.74)
+		(stroke
+			(width 0.2032)
+			(type solid)
+		)
+		(fill no)
+		(layer "User.1")
+	)
+	(gr_text "In the box I made, the routings not great, a lot of places have vias where they dont need if the\nrouting and placement was done better. An example of this is the resistor for the transciever (RRS4?)\nIs super far away from the transciever so it leads to you using vias where not needed\n\nyou should have a 10uf at the 24V input header, also you should move it further from the hbridge since the \nheatsink will overlap, if you turn on silkscreen you should see it\n\nif smth is tht and connected to GND, it doesnt need a via\n\nSuper important: ur constraints are not set up right, so it might show that it \npasses the DRC, but the DRC is just wrong if the constraints are wrong\n\nlater:\nclean up silkscreen, add pinouts on the silkscreen\n"
+		(at 92.08 35.71 0)
+		(layer "User.1")
+		(effects
+			(font
+				(size 1 1)
+				(thickness 0.15)
+			)
+			(justify left bottom)
+		)
 	)
 	(segment

Commit message: intl fixes
Parts:
- moved RRS4 23.6 mm to (145.3, 61.7), turned to 0 degrees
- moved CVin1 9.59 mm to (115.6, 79.5)
- moved RRS3 6.89 mm to (152.4, 60.2), turned to 180 degrees
- moved RRS2 5.80 mm to (149.9, 60.2), turned to 180 degrees
- moved J5 3.49 mm to (108.0, 85.7)
- moved CRS1 3.30 mm to (139.7, 59.7)
- moved RRS6 2.03 mm to (144.5, 63.5)
- moved RRS5 2.03 mm to (145.8, 63.5)
Routing:
- net Net-(J12-Pin_2): track 59.5 -> 39.0 mm, vias 2 -> 4
- net Net-(J12-Pin_3): track 29.6 -> 34.7 mm, vias 6 -> 4
- net +24V: track 84.1 -> 88.3 mm
- net GND: track 63.2 -> 59.0 mm, vias 30 -> 28
- net +5V: track 125.8 -> 122.5 mm
- net +3.3V: track 87.6 -> 89.9 mm
- net /52: track 17.4 -> 15.5 mm
- net /51: vias 2 -> 4
Other:
- board text added: "In the box I made, the routings not great, a lot of places have vias where they dont need if the routing and placement was done better. An example of this is the resistor for the transciever (RRS4?)--ok Is super far away from the transciever so it leads to you using vias where not needed -- ok you should have a 10uf at the 24V input header, also you should move it further from the hbridge since t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"
- board text removed: "In the box I made, the routings not great, a lot of places have vias where they dont need if the routing and placement was done better. An example of this is the resistor for the transciever (RRS4?) Is super far away from the transciever so it leads to you using vias where not needed you should have a 10uf at the 24V input header, also you should move it further from the hbridge since the heatsin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"

Commit message: review2
Routing:
- net GND: track 59.0 -> 49.1 mm, vias 28 -> 23
- net +3.3V: track 89.9 -> 89.2 mm
Other:
- board text added: "RUN DRC, you are missing some ground VIAS Vias go through layers, throughhole components already go thgrough the layers If you look at the shaded blue part, you'll see theres no {dblquote}bubble{dblquote} around tht components that need ground, there is a t shape through them, so they are already connected to ground. Only surface mount pads need them since they need some way to get the ground con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"
Changed lines of the file:
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@@
 		(layer "Edge.Cuts")
+	)
+	(gr_text "RUN DRC, you are missing some ground VIAS\n\nVias go through layers, throughhole components already go thgrough the layers\nIf you look at the shaded blue part, you'll see theres no {dblquote}bubble{dblquote} around\ntht components that need ground, there is a t shape through them, so they are\nalready connected to ground. Only surface mount pads need them since they\nneed some way to get the ground connection\n\nthe traces going to the motor should be much much thicker, the traces\nThe traces going to the servos and any high current carrying routes\nshould be thicker as well. Similalry if you have a wider trace, you need \na wider via, the via hole should = trace width, and the via diamter should be double\nalso if you have a capacitor with a thick power trace, the ground trace\nshould be equally as thick\n\nConstraints are in the board setup tab... also google... :(\n\nclean up silkscreen by removing the stuff u dont need and putting\nhelpful labels that will make it easy to assemble and use"
+		(at 99.51 142.1 0)
+		(layer "F.Cu")
+		(effects
+			(font
+				(size 1.5 1.5)
+				(thickness 0.3)
+				(bold yes)
+			)
+			(justify left bottom)
+		)
 	)
 	(gr_text "In the box I made, the routings not great, a lot of places have vias where they dont need if the\nrouting and placement was done better. An example of this is the resistor for the transciever (RRS4?)--ok\nIs super far away from the transciever so it leads to you using vias where not needed -- ok\n\nyou should have a 10uf at the 24V input header, also you should move it further from the hbridge since the \nheatsink will overlap, if you turn on silkscreen you should see it -- ok\n\nif smth is tht and connected to GND, it doesnt need a via -- plz clarify i thought u needed to connect everything to gnd via vias\n\nSuper important: ur constraints are not set up right, so it might show that it \npasses the DRC, but the DRC is just wrong if the constraints are wrong\n-- how do i setup constraints\n\nlater:\nclean up silkscreen, add pinouts on the silkscreen\n-- how do i clean up silkscreen "
@@
 	)
 	(segment
-		(start 127.6483 64.6081)
-		(end 127.6483 64.32)
+		(start 121.559 68.072)
+		(end 124.1104 65.5206)
 		(width 0.2)
 		(layer "F.Cu")
@@
 	)
 	(segment
-		(start 128.8 64.32)
-		(end 127.6483 64.32)
+		(start 126.7358 65.5206)
+		(end 127.9364 64.32)
 		(width 0.2)
 		(layer "F.Cu")
@@
 	)
 	(segment
-		(start 121.559 68.072)
-		(end 124.1104 65.5206)
-		(width 0.2)
-		(layer "F.Cu")
-		(net 14)
-	)
-	(segment
-		(start 126.7358 65.5206)
-		(end 127.6483 64.6081)
+		(start 127.9364 64.32)
+		(end 128.8 64.32)
 		(width 0.2)
 		(layer "F.Cu")
@@
 	)
 	(segment
-		(start 151.66 56.67)
-		(end 151.66 58.652)
-		(width 0.2)
-		(layer "F.Cu")
-		(net 15)
-	)
-	(segment
 		(start 141.986 66.294)
 		(end 141.732 66.548)
@@
 	)
 	(segment
-		(start 151.66 58.652)
-		(end 151.638 58.674)
-		(width 0.2)
-		(layer "F.Cu")
-		(net 15)
-	)
-	(segment
 		(start 139.2135 67.564)
 		(end 139.2135 68.6015)
@@
 	)
 	(segment
-		(start 121.559 75.692)
-		(end 123.444 75.692)
-		(width 0.2)
-		(layer "F.Cu")
-		(net 15)
-	)
-	(segment
 		(start 131.064 52.324)
 		(end 132.08 51.308)
@@
 	)
 	(segment
-		(start 121.559 57.912)
-		(end 122.829 56.642)
-		(width 0.2)
-		(layer "F.Cu")
-		(net 15)
-	)
-	(segment
 		(start 110.33 51.308)
 		(end 110.33 53.754)
@@
 	)
 	(segment
-		(start 126.746 77.47)
-		(end 127.254 76.962)
-		(width 0.2)
-		(layer "F.Cu")
-		(net 15)
-	)
-	(segment
 		(start 119.1045 52.324)
 		(end 119.1045 53.8695)
@@
 	)
 	(segment
-		(start 125.984 77.47)
-		(end 126.746 77.47)
-		(width 0.2)
-		(layer "F.Cu")
-		(net 15)
-	)
-	(segment
-		(start 125.73 51.308)
-		(end 125.476 51.562)
-		(width 0.2)
-		(layer "F.Cu")
-		(net 15)
-	)
-	(segment
-		(start 125.73 49.784)
-		(end 125.73 51.308)
-		(width 0.2)
-		(layer "F.Cu")
-		(net 15)
-	)
-	(segment
 		(start 139.2135 68.6015)
 		(end 139.7 69.088)
@@
 	)
 	(segment
-		(start 122.829 56.642)
-		(end 123.698 56.642)
-		(width 0.2)
-		(layer "F.Cu")
-		(net 15)
-	)
-	(segment
 		(start 132.716 73.406)
 		(end 132.716 72.008)
@@
 	)
 	(via
-		(at 125.476 51.562)
-		(size 0.6)
-		(drill 0.3)
-		(layers "F.Cu" "B.Cu")
-		(net 15)
-	)
-	(via
 		(at 135.89 84.328)
 		(size 0.6)
@@
 	)
 	(via
-		(at 123.444 75.692)
-		(size 0.6)
-		(drill 0.3)
-		(layers "F.Cu" "B.Cu")
-		(net 15)
-	)
-	(via
 		(at 141.986 73.66)
 		(size 0.6)
@@
 	)
 	(via
-		(at 123.698 56.642)
-		(size 0.6)
-		(drill 0.3)
-		(layers "F.Cu" "B.Cu")
-		(net 15)
-	)
-	(via
 		(at 126.492 89.662)
 		(size 0.6)
@@
 	)
 	(via
-		(at 151.638 58.674)
-		(size 0.6)
-		(drill 0.3)
-		(layers "F.Cu" "B.Cu")
-		(net 15)
-	)
-	(via
 		(at 137.414 69.342)
 		(size 0.6)
@@
 	(via
 		(at 150.368 48.514)
-		(size 0.6)
-		(drill 0.3)
-		(layers "F.Cu" "B.Cu")
-		(net 15)
-	)
-	(via
-		(at 127.254 76.962)
 		(size 0.6)
 		(drill 0.3)
@@
 	)
 	(segment
+		(start 152.7638 65.7338)
+		(end 152.7638 66.7198)
+		(width 0.5)
+		(layer "F.Cu")
+		(net 28)
+	)
+	(segment
+		(start 146.394913 64.0975)
+		(end 145.796 64.0975)
+		(width 0.5)
+		(layer "F.Cu")
+		(net 28)
+	)
+	(segment
+		(start 149.8423 83.911)
+		(end 149.3353 84.418)
+		(width 0.5)
+		(layer "F.Cu")
+		(net 28)
+	)
+	(segment
+		(start 147.156913 64.8595)
+		(end 146.394913 64.0975)
+		(width 0.5)
+		(layer "F.Cu")
+		(net 28)
+	)
+	(segment
 		(start 147.828 64.8595)
 		(end 148.0893 64.5982)
@@
 	)
 	(segment
-		(start 146.394913 64.0975)
-		(end 145.796 64.0975)
-		(width 0.5)
-		(layer "F.Cu")
-		(net 28)
-	)
-	(segment
-		(start 149.8423 83.911)
-		(end 149.3353 84.418)
-		(width 0.5)
-		(layer "F.Cu")
-		(net 28)
-	)
-	(segment
-		(start 147.156913 64.8595)
-		(end 146.394913 64.0975)
+		(start 151.6282 64.5982)
+		(end 152.7638 65.7338)
 		(width 0.5)
 		(layer "F.Cu")
@@
 	)
 	(segment
+		(start 153.924 81.788)
+		(end 153.924 67.88)
+		(width 0.5)
+		(layer "F.Cu")
+		(net 28)
+	)
+	(segment
+		(start 147.109 66.7805)
+		(end 147.32 66.7805)
+		(width 0.5)
+		(layer "F.Cu")
+		(net 28)
+	)
+	(segment
+		(start 144.4215 90.819)
+		(end 148.941 86.2995)
+		(width 0.5)
+		(layer "F.Cu")
+		(net 28)
+	)
+	(segment
+		(start 148.0893 64.5982)
+		(end 151.6282 64.5982)
+		(width 0.5)
+		(layer "F.Cu")
+		(net 28)
+	)
+	(segment
+		(start 125.829 90.819)
+		(end 144.4215 90.819)
+		(width 0.5)
+		(layer "F.Cu")
+		(net 28)
+	)
+	(segment
+		(start 147.828 66.2236)
+		(end 147.828 64.8595)
+		(width 0.5)
+		(layer "F.Cu")
+		(net 28)
+	)
+	(segment
+		(start 151.039 83.911)
+		(end 152.4 82.55)
+		(width 0.5)
+		(layer "F.Cu")
+		(net 28)
+	)
+	(segment
 		(start 152.7638 66.7198)
 		(end 153.035 66.991)
@@
 	)
 	(segment
-		(start 153.924 81.788)
-		(end 153.924 67.88)
-		(width 0.5)
-		(layer "F.Cu")
-		(net 28)
-	)
-	(segment
-		(start 152.7638 64.5982)
-		(end 152.7638 66.7198)
-		(width 0.5)
-		(layer "F.Cu")
-		(net 28)
-	)
-	(segment
-		(start 147.109 66.7805)
-		(end 147.32 66.7805)
-		(width 0.5)
-		(layer "F.Cu")
-		(net 28)
-	)
-	(segment
-		(start 144.4215 90.819)
-		(end 148.941 86.2995)
-		(width 0.5)
-		(layer "F.Cu")
-		(net 28)
-	)
-	(segment
-		(start 125.829 90.819)
-		(end 144.4215 90.819)
-		(width 0.5)
-		(layer "F.Cu")
-		(net 28)
-	)
-	(segment
-		(start 147.828 66.2236)
-		(end 147.828 64.8595)
-		(width 0.5)
-		(layer "F.Cu")
-		(net 28)
-	)
-	(segment
-		(start 151.039 83.911)
-		(end 152.4 82.55)
-		(width 0.5)
-		(layer "F.Cu")
-		(net 28)
-	)
-	(segment
 		(start 146.8335 66.294)
 		(end 147.32 66.7805)
@@
 	)
 	(segment
-		(start 148.0893 64.5982)
-		(end 152.7638 64.5982)
-		(width 0.5)
-		(layer "F.Cu")
-		(net 28)
-	)
-	(segment
 		(start 148.941 86.308)
 		(end 148.941 85.78)
@@
 	)
 	(segment
+		(start 144.348 78.1117)
+		(end 145.2117 78.9754)
+		(width 0.2)
+		(layer "F.Cu")
+		(net 44)
+	)
+	(segment
+		(start 144.06 76.96)
+		(end 144.06 77.81)
+		(width 0.2)
+		(layer "F.Cu")
+		(net 44)
+	)
+	(segment
+		(start 144.06 77.81)
+		(end 144.348 78.098)
+		(width 0.2)
+		(layer "F.Cu")
+		(net 44)
+	)
+	(segment
+		(start 145.2117 79.8315)
+		(end 146.441 81.0608)
+		(width 0.2)
+		(layer "F.Cu")
+		(net 44)
+	)
+	(segment
+		(start 144.348 78.098)
+		(end 144.348 78.1117)
+		(width 0.2)
+		(layer "F.Cu")
+		(net 44)
+	)
+	(segment
 		(start 145.2117 78.9754)
 		(end 145.2117 79.8315)
@@
 	)
 	(segment
-		(start 144.06 76.96)
-		(end 144.06 78.1117)
-		(width 0.2)
-		(layer "F.Cu")
-		(net 44)
-	)
-	(segment
-		(start 144.348 78.1117)
-		(end 145.2117 78.9754)
-		(width 0.2)
-		(layer "F.Cu")
-		(net 44)
-	)
-	(segment
 		(start 146.441 81.0608)
 		(end 146.441 85.78)
 		(width 0.2)
 		(layer "F.Cu")
-		(net 44)
-	)
-	(segment
-		(start 144.06 78.1117)
-		(end 144.348 78.1117)
-		(width 0.2)
-		(layer "F.Cu")
-		(net 44)
-	)
-	(segment
-		(start 145.2117 79.8315)
-		(end 146.441 81.0608)
-		(width 0.2)
-		(layer "F.Cu")
