File: PCBs/2Dof/2Dof.kicad_sch (KiCad schematic)
At the start: 50 parts, among them J1 Conn_02x07_Odd_Even, J12 RS485, J14 HBA, J17 Servo1, J2 Conn_02x08_Odd_Even, J3 Conn_02x08_Odd_Even, J5 24Vin, J9 Laser Diode, Q1 QServoA, Q6 LaserDiodeT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

Commit message: review2
Other:
- note added: "for the transistor stuff, put the capacitors on the output by the headers instead (same for servo)"
Changed lines of the file:
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@@
 	(generator_version "9.0")
 	(paper "A4")
+	(text "for the transistor stuff, put the capacitors on the output by the headers instead\n(same for servo)"
+		(exclude_from_sim no)
+		(at 101.854 98.552 0)
+		(effects
+			(font
+				(size 1.27 1.27)
+			)
+		)
+	)
 	(text_box "Laser Diode"
 		(exclude_from_sim no)
