File: PCBs/2Dof/2Dof-tests.kicad_pcb (KiCad board)
At the start: 2 copper layers, 54.4 x 47 mm, 48 parts, among them J1 Conn_02x07_Odd_Even, J12 RS485, J14 HBA, J17 Servo1, J2 Conn_02x08_Odd_Even, J3 Conn_02x08_Odd_Even, J9 Laser Diode, Q1 QServoA, Q6 LaserDiodeT, U1 MAX485E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

Commit message: final (i think)
Parts:
- moved 24Vin 3.89 mm to (108.2, 86.7), turned to 0 degrees
Routing:
- net +24V: track 64.2 -> 67.3 mm
- net /41: track 24.6 -> 25.1 mm
- net GND: track 53.0 -> 53.1 mm, vias 21 -> 22
Other:
- board size 54.4 x 47 mm -> 54.4 x 48 mm
- board text added: "M1"
- board text added: "PWM"
- board text added: "Sig"
- board text added: "VSS"
- board text added: "Vin"
- board text removed: "AMT"
- board text removed: "DC"
- board text removed: "like this"
- board text removed: "or liek this"
- board text removed: "what do i even do for pinouts?"
