File: PCBs/2Dof/2Dof-tests.kicad_pcb (KiCad board)
At the start: 2 copper layers, 54.4 x 48 mm, 48 parts, among them J1 Conn_02x07_Odd_Even, J12 RS485, J14 HBA, J17 Servo1, J2 Conn_02x08_Odd_Even, J3 Conn_02x08_Odd_Even, J9 Laser Diode, Q1 QServoA, Q6 LaserDiodeT, U1 MAX485E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

Commit message: fixes :(((((((
Parts:
- moved J5 3.86 mm to (109.9, 83.2), turned to 90 degrees
- renumbered 24Vin to J5
Connections:
- J5 pad 1: +24V -> GND
- J5 pad 2: GND -> +24V
Routing:
- net +24V: track 67.3 -> 61.9 mm
Changed lines of the file:
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@@
 	(footprint "Connector_Molex:Molex_Micro-Fit_3.0_43045-0200_2x01_P3.00mm_Horizontal"
 		(layer "F.Cu")
-		(at 108.204 86.659)
+		(at 109.94 83.21 90)
 		(descr "Molex Micro-Fit 3.0 Connector System, 43045-0200 (alternative finishes: 43045-020x), 1 Pins per row (https://www.molex.com/pdm_docs/sd/430450201_sd.pdf), generated with kicad-footprint-generator")
 		(tags "connector Molex Micro-Fit_3.0 horizontal")
-		(property "Reference" "24Vin"
-			(at 5.08 -4.572 90)
+		(property "Reference" "J5"
+			(at 5.08 -4.572 0)
 			(layer "F.SilkS")
 			(effects
@@
 		)
 		(property "Value" "24Vin"
-			(at 0 5.7 0)
+			(at 0 5.7 90)
 			(layer "F.Fab")
 			(effects
@@
 		)
 		(property "Datasheet" "~"
-			(at 0 0 0)
+			(at 0 0 90)
 			(layer "F.Fab")
 			(hide yes)
@@
 		)
 		(property "Description" "Generic connector, single row, 01x02, script generated (kicad-library-utils/schlib/autogen/connector/)"
-			(at 0 0 0)
+			(at 0 0 90)
 			(layer "F.Fab")
 			(hide yes)
@@
 		(attr through_hole)
 		(fp_line
-			(start -3.685 -8.03)
-			(end -2.685 -9.03)
+			(start 2.685 -9.03)
+			(end 3.685 -8.03)
 			(stroke
 				(width 0.12)
@@
 		)
 		(fp_line
-			(start -3.685 1.1)
-			(end -3.685 -8.03)
+			(start -2.685 -9.03)
+			(end 2.685 -9.03)
 			(stroke
 				(width 0.12)
@@
 		)
 		(fp_line
-			(start -2.685 -9.03)
-			(end 2.685 -9.03)
+			(start 3.685 -8.03)
+			(end 3.685 1.1)
 			(stroke
 				(width 0.12)
@@
 		)
 		(fp_line
-			(start 2.685 -9.03)
-			(end 3.685 -8.03)
+			(start -3.685 -8.03)
+			(end -2.685 -9.03)
 			(stroke
 				(width 0.12)
@@
 		)
 		(fp_line
-			(start 3.685 -8.03)
-			(end 3.685 1.1)
+			(start 3.685 1.1)
+			(end -3.685 1.1)
 			(stroke
 				(width 0.12)
@@
 		)
 		(fp_line
-			(start 3.685 1.1)
-			(end -3.685 1.1)
+			(start -3.685 1.1)
+			(end -3.685 -8.03)
 			(stroke
 				(width 0.12)
@@
 		)
 		(fp_line
-			(start -4.08 -9.42)
-			(end 4.08 -9.42)
+			(start 4.08 -9.42)
+			(end 4.08 1.5)
 			(stroke
 				(width 0.05)
@@
 		)
 		(fp_line
-			(start -4.08 1.5)
-			(end -4.08 -9.42)
+			(start -4.08 -9.42)
+			(end 4.08 -9.42)
 			(stroke
 				(width 0.05)
@@
 		)
 		(fp_line
-			(start -1.25 1.5)
-			(end -4.08 1.5)
+			(start 4.08 1.5)
+			(end 1.25 1.5)
 			(stroke
 				(width 0.05)
@@
 		)
 		(fp_line
-			(start -1.25 4.25)
-			(end -1.25 1.5)
+			(start 1.25 1.5)
+			(end 1.25 4.25)
 			(stroke
 				(width 0.05)
@@
 		)
 		(fp_line
-			(start 1.25 1.5)
-			(end 1.25 4.25)
+			(start -1.25 1.5)
+			(end -4.08 1.5)
 			(stroke
 				(width 0.05)
@@
 		)
 		(fp_line
-			(start 1.25 4.25)
-			(end -1.25 4.25)
+			(start -4.08 1.5)
+			(end -4.08 -9.42)
 			(stroke
 				(width 0.05)
@@
 		)
 		(fp_line
-			(start 4.08 -9.42)
-			(end 4.08 1.5)
+			(start 1.25 4.25)
+			(end -1.25 4.25)
 			(stroke
 				(width 0.05)
@@
 		)
 		(fp_line
-			(start 4.08 1.5)
-			(end 1.25 1.5)
+			(start -1.25 4.25)
+			(end -1.25 1.5)
 			(stroke
 				(width 0.05)
@@
 		)
 		(fp_line
-			(start -3.575 -7.92)
-			(end -2.575 -8.92)
+			(start 2.575 -8.92)
+			(end 3.575 -7.92)
 			(stroke
 				(width 0.1)
@@
 		)
 		(fp_line
-			(start -3.575 0.99)
-			(end -3.575 -7.92)
+			(start -2.575 -8.92)
+			(end 2.575 -8.92)
 			(stroke
 				(width 0.1)
@@
 		)
 		(fp_line
-			(start -2.575 -8.92)
-			(end 2.575 -8.92)
+			(start 3.575 -7.92)
+			(end 3.575 0.99)
 			(stroke
 				(width 0.1)
@@
 		)
 		(fp_line
-			(start -0.75 0.99)
-			(end 0 0)
+			(start -3.575 -7.92)
+			(end -2.575 -8.92)
 			(stroke
 				(width 0.1)
@@
 		)
 		(fp_line
-			(start 2.575 -8.92)
-			(end 3.575 -7.92)
+			(start 3.575 0.99)
+			(end -3.575 0.99)
 			(stroke
 				(width 0.1)
@@
 		)
 		(fp_line
-			(start 3.575 -7.92)
-			(end 3.575 0.99)
+			(start -0.75 0.99)
+			(end 0 0)
 			(stroke
 				(width 0.1)
@@
 		)
 		(fp_line
-			(start 3.575 0.99)
-			(end -3.575 0.99)
+			(start -3.575 0.99)
+			(end -3.575 -7.92)
 			(stroke
 				(width 0.1)
@@
 		)
 		(fp_text user "${REFERENCE}"
-			(at 0 -8.22 0)
+			(at 0 -8.22 90)
 			(layer "F.Fab")
 			(effects
@@
 		)
 		(pad "" np_thru_hole circle
-			(at 0 -4.32)
+			(at 0 -4.32 90)
 			(size 3 3)
 			(drill 3)
@@
 		)
 		(pad "1" thru_hole roundrect
-			(at 0 0)
+			(at 0 0 90)
 			(size 1.5 1.5)
 			(drill 1.02)
@@
 			(remove_unused_layers no)
 			(roundrect_rratio 0.166667)
-			(net 47 "+24V")
+			(net 15 "GND")
 			(pinfunction "Pin_1")
 			(pintype "passive")
 		)
 		(pad "2" thru_hole circle
-			(at 0 3)
+			(at 0 3 90)
 			(size 1.5 1.5)
 			(drill 1.02)
 			(layers "*.Cu" "*.Mask")
 			(remove_unused_layers no)
-			(net 15 "GND")
+			(net 47 "+24V")
 			(pinfunction "Pin_2")
 			(pintype "passive")
@@
 	)
 	(segment
+		(start 112.94 81.923)
+		(end 113.837 81.026)
+		(width 1)
+		(layer "F.Cu")
+		(net 47)
+	)
+	(segment
 		(start 115.651 80.853)
 		(end 115.824 81.026)
@@
 	)
 	(segment
+		(start 112.94 83.21)
+		(end 112.94 81.923)
+		(width 1)
+		(layer "F.Cu")
+		(net 47)
+	)
+	(segment
 		(start 116.0565 78.994)
 		(end 115.64 78.5775)
@@
 		(width 1)
 		(layer "F.Cu")
-		(net 47)
-	)
-	(segment
-		(start 113.837 81.026)
-		(end 108.204 86.659)
-		(width 1)
-		(layer "F.Cu")
