File: PCBs/2Dof/2Dof-tests.kicad_sch (KiCad schematic)
At the start: 50 parts, among them J1 Conn_02x07_Odd_Even, J12 RS485, J14 HBA, J17 Servo1, J2 Conn_02x08_Odd_Even, J3 Conn_02x08_Odd_Even, J5 24Vin, J9 Laser Diode, Q1 QServoA, Q6 LaserDiodeT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

Commit message: fixes :(((((((
Connections:
- net +24V: now also J5.2 (Pin_2); no longer J5.1 (Pin_1)
- net GND: now also J5.1 (Pin_1); no longer J5.2 (Pin_2)
Changed lines of the file:
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@@
 	(symbol
 		(lib_id "Connector_Generic:Conn_01x02")
-		(at 45.72 167.64 0)
+		(at 45.72 170.18 0)
+		(mirror x)
 		(unit 1)
 		(exclude_from_sim no)
@@
 		(on_board yes)
 		(dnp no)
-		(fields_autoplaced yes)
 		(property "Reference" "J5"
-			(at 48.26 167.6399 0)
+			(at 48.26 170.1801 0)
 			(effects
 				(font
@@
 		)
 		(property "Value" "24Vin"
-			(at 48.26 170.1799 0)
+			(at 48.26 167.6401 0)
 			(effects
 				(font
@@
 		)
 		(property "Footprint" "Connector_Molex:Molex_Micro-Fit_3.0_43045-0200_2x01_P3.00mm_Horizontal"
-			(at 45.72 167.64 0)
+			(at 45.72 170.18 0)
 			(effects
 				(font
@@
 		)
 		(property "Datasheet" "~"
-			(at 45.72 167.64 0)
+			(at 45.72 170.18 0)
 			(effects
 				(font
@@
 		)
 		(property "Description" "Generic connector, single row, 01x02, script generated (kicad-library-utils/schlib/autogen/connector/)"
-			(at 45.72 167.64 0)
+			(at 45.72 170.18 0)
 			(effects
 				(font
