File: PCBs/Fluoro_PCB/Fluoro_PCB/Fluoro_PCB.kicad_pcb (KiCad board)
At the start: 2 copper layers, 45.5 x 32.5 mm, 14 parts, among them J1 Conn_02x07_Odd_Even, J2 Conn_02x08_Odd_Even, J3 Conn_02x08_Odd_Even, J4 Conn_01x02_Pin, J5 Conn_01x02_Pin, Q1 S8050, Q2 S8550, U1 OPT101P

Commit message: Add files via upload
Parts:
- added C2: 100uF, Capacitor_SMD:C_0201_0603Metric, F.Cu at (143.0, 63.9)
Connections:
- R2 pad 1: Net-(U1-OUTPUT) -> Net-(U1-1MOHM_FB)
- U1 pad 4: unconnected-(U1-1MOHM_FB-Pad4) -> Net-(U1-1MOHM_FB)
- U1 pad 5: Net-(U1-OUTPUT) -> Net-(U1-1MOHM_FB)
Routing:
- net Net-(U1-OUTPUT): track 3.81 -> 0.00 mm
- net Net-(U1-1MOHM_FB): track 0.00 -> 3.81 mm
- net GND: track 18.7 -> 22.4 mm
- net +5V: track 12.0 -> 13.5 mm
