File: PCBs/Fluoro_PCB/Fluoro_PCB/Fluoro_PCB.kicad_pcb (KiCad board)
At the start: 2 copper layers, 38.8 x 31.2 mm, 21 parts, among them J1 Conn_02x07_Odd_Even, J2 Conn_02x08_Odd_Even, J3 Conn_02x08_Odd_Even, J4 SM02B-GHS-TB, J6 SM02B-GHS-TB, Q1 S8050, Q2 S8550, U1 OPT101P

Commit message: delete redudant vias
Routing:
- net GND: track 18.5 -> 13.9 mm, vias 6 -> 3
Changed lines of the file:
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@@
-	)
-	(segment
-		(start 151.66 56.67)
-		(end 153.92 56.67)
-		(width 0.2)
-		(layer "F.Cu")
-		(net 15)
-	)
-	(segment
-		(start 132.37 59.62)
-		(end 132 59.25)
-		(width 0.2)
-		(layer "F.Cu")
-		(net 15)
 	)
 	(segment
 		(start 155.825 62.2)
 		(end 155.9 62.125)
-		(width 0.2)
-		(layer "F.Cu")
-		(net 15)
-	)
-	(segment
-		(start 132.37 60.96)
-		(end 132.37 59.62)
-		(width 0.2)
-		(layer "F.Cu")
-		(net 15)
-	)
-	(segment
-		(start 153.92 56.67)
-		(end 154.25 57)
 		(width 0.2)
 		(layer "F.Cu")
@@
 	)
 	(via
-		(at 154.25 57)
-		(size 0.6)
-		(drill 0.3)
-		(layers "F.Cu" "B.Cu")
-		(free yes)
-		(net 15)
-	)
-	(via
 		(at 152.75 63.75)
-		(size 0.6)
-		(drill 0.3)
-		(layers "F.Cu" "B.Cu")
-		(free yes)
-		(net 15)
-	)
-	(via
-		(at 154.25 57)
 		(size 0.6)
 		(drill 0.3)
@@
 		(size 0.6)
 		(drill 0.3)
-		(layers "F.Cu" "B.Cu")
-		(free yes)
-		(net 15)
-	)
-	(via
-		(at 132 59.25)
-		(size 0.6)
-		(drill 0.3)
