File: PCBs/Fluoro_PCB/Fluoro_PCB/Fluoro_PCB.kicad_sch (KiCad schematic)
At the start: 14 parts, among them J1 Conn_02x07_Odd_Even, J2 Conn_02x08_Odd_Even, J3 Conn_02x08_Odd_Even, J4 Conn_01x02_Pin, J5 Conn_01x02_Pin, Q1 S8050, Q2 S8550, U1 OPT101P

Commit message: Add files via upload
Parts:
- added C2: 100uF, Capacitor_SMD:C_0201_0603Metric, symbol Device:C
Connections:
- net +5V: now also C2.2
- net GND: now also C2.1
- net at R2.1, U1.5 (OUTPUT): now also U1.4 (1MOHM_FB)
Changed lines of the file:
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@@
+	)
+	(junction
+		(at 177.8 72.39)
+		(diameter 0)
+		(color 0 0 0 0)
 	)
 	(junction
@@
 	)
 	(junction
+		(at 185.42 64.77)
+		(diameter 0)
+		(color 0 0 0 0)
+	)
+	(junction
 		(at 170.18 22.86)
 		(diameter 0)
@@
 	(wire
 		(pts
+			(xy 139.7 72.39) (xy 133.35 72.39)
+		)
+		(stroke
+			(width 0)
+			(type default)
+		)
+	)
+	(wire
+		(pts
 			(xy 134.62 120.65) (xy 134.62 105.41)
 		)
@@
 	(wire
 		(pts
+			(xy 133.35 86.36) (xy 177.8 86.36)
+		)
+		(stroke
+			(width 0)
+			(type default)
+		)
+	)
+	(wire
+		(pts
 			(xy 170.18 22.86) (xy 179.07 22.86)
 		)
@@
 	(wire
 		(pts
+			(xy 194.31 64.77) (xy 185.42 64.77)
+		)
+		(stroke
+			(width 0)
+			(type default)
+		)
+	)
+	(wire
+		(pts
 			(xy 119.38 52.07) (xy 119.38 59.69)
 		)
@@
 	(wire
 		(pts
+			(xy 185.42 64.77) (xy 175.26 64.77)
+		)
+		(stroke
+			(width 0)
+			(type default)
+		)
+	)
+	(wire
+		(pts
+			(xy 177.8 86.36) (xy 177.8 72.39)
+		)
+		(stroke
+			(width 0)
+			(type default)
+		)
+	)
+	(wire
+		(pts
 			(xy 168.91 22.86) (xy 170.18 22.86)
 		)
@@
 	(wire
 		(pts
-			(xy 175.26 72.39) (xy 184.15 72.39)
+			(xy 175.26 72.39) (xy 177.8 72.39)
 		)
 		(stroke
@@
 	(wire
 		(pts
+			(xy 177.8 72.39) (xy 184.15 72.39)
+		)
+		(stroke
+			(width 0)
+			(type default)
+		)
+	)
+	(wire
+		(pts
 			(xy 204.47 77.47) (xy 204.47 74.93)
 		)
@@
 		(pts
 			(xy 128.27 52.07) (xy 119.38 52.07)
+		)
+		(stroke
+			(width 0)
+			(type default)
+		)
+	)
+	(wire
+		(pts
+			(xy 133.35 72.39) (xy 133.35 86.36)
 		)
 		(stroke
@@
 	)
 	(symbol
+		(lib_id "OPT101P:GND")
+		(at 185.42 57.15 180)
+		(unit 1)
+		(exclude_from_sim no)
+		(in_bom yes)
+		(on_board yes)
+		(dnp no)
+		(fields_autoplaced yes)
+		(property "Reference" "#PWR05"
+			(at 185.42 50.8 0)
+			(effects
+				(font
+					(size 1.27 1.27)
+				)
+				(hide yes)
+			)
+		)
+		(property "Value" "GND"
+			(at 185.42 52.07 0)
+			(effects
+				(font
+					(size 1.27 1.27)
+				)
+			)
+		)
+		(property "Footprint" ""
+			(at 185.42 57.15 0)
+			(effects
+				(font
+					(size 1.27 1.27)
+				)
+				(hide yes)
+			)
+		)
+		(property "Datasheet" ""
+			(at 185.42 57.15 0)
+			(effects
+				(font
+					(size 1.27 1.27)
+				)
+				(hide yes)
+			)
+		)
+		(property "Description" "Power symbol creates a global label with name \"GND\" , ground"
+			(at 185.42 57.15 0)
+			(effects
+				(font
+					(size 1.27 1.27)
+				)
+				(hide yes)
+			)
+		)
+		(pin "1"
+		)
+		(instances
+			(project "Fluoro_PCB"
+				(path "/705004fe-9694-4831-a243-8c72357320a8"
+					(reference "#PWR05")
+					(unit 1)
+				)
+			)
+		)
+	)
+	(symbol
 		(lib_id "OPT101P:+15V")
-		(at 175.26 64.77 270)
+		(at 194.31 64.77 270)
 		(unit 1)
 		(exclude_from_sim no)
@@
 		(fields_autoplaced yes)
 		(property "Reference" "#PWR0101"
-			(at 171.45 64.77 0)
+			(at 190.5 64.77 0)
 			(effects
 				(font
@@
 		)
 		(property "Value" "+5V"
-			(at 179.07 64.7699 90)
+			(at 198.12 64.7699 90)
 			(effects
 				(font
@@
 		)
 		(property "Footprint" ""
-			(at 175.26 64.77 0)
+			(at 194.31 64.77 0)
 			(effects
 				(font
@@
 		)
 		(property "Datasheet" ""
-			(at 175.26 64.77 0)
+			(at 194.31 64.77 0)
 			(effects
 				(font
@@
 		)
 		(property "Description" "Power symbol creates a global label with name \"+15V\""
-			(at 175.26 64.77 0)
+			(at 194.31 64.77 0)
 			(effects
 				(font
@@
 					(unit 1)
 				)
+			)
+		)
+	)
+	(symbol
+		(lib_id "Device:C")
+		(at 185.42 60.96 0)
+		(unit 1)
+		(exclude_from_sim no)
+		(in_bom yes)
+		(on_board yes)
+		(dnp no)
+		(fields_autoplaced yes)
+		(property "Reference" "C2"
+			(at 189.23 59.6899 0)
+			(effects
+				(font
+					(size 1.27 1.27)
+				)
+				(justify left)
+			)
+		)
+		(property "Value" "100uF"
+			(at 189.23 62.2299 0)
+			(effects
+				(font
+					(size 1.27 1.27)
+				)
+				(justify left)
+			)
+		)
+		(property "Footprint" "Capacitor_SMD:C_0201_0603Metric"
+			(at 186.3852 64.77 0)
+			(effects
+				(font
+					(size 1.27 1.27)
+				)
+				(hide yes)
+			)
+		)
+		(property "Datasheet" "~"
+			(at 185.42 60.96 0)
+			(effects
+				(font
+					(size 1.27 1.27)
+				)
+				(hide yes)
+			)
+		)
+		(property "Description" "Unpolarized capacitor"
+			(at 185.42 60.96 0)
+			(effects
+				(font
+					(size 1.27 1.27)
+				)
+				(hide yes)
+			)
+		)
+		(pin "2"
+		)
+		(pin "1"
+		)
+		(instances
+			(project "Fluoro_PCB"
+				(path "/705004fe-9694-4831-a243-8c72357320a8"
+					(reference "C2")
+					(unit 1)
+				)
