File: PCBs/Fluoro_PCB/Fluoro_PCB.kicad_sch (KiCad schematic)
At the start: 12 parts, among them J1 Conn_02x07_Odd_Even, J2 Conn_02x08_Odd_Even, J3 Conn_02x08_Odd_Even, J4 Conn_01x02_Pin, J5 Conn_01x02_Pin, U1 OPT101P, U3 LM393N

Commit message: Add files via upload
Parts:
- removed R4: 10000, Resistor_SMD:R_0201_0603Metric, symbol OPT101P:R
- removed U3: LM393N, LM393N_NOPB:DIP794W45P254L959H508Q8, symbol OPT101P:LM393N
- added Q1: S8050, Package_TO_SOT_THT:TO-92_Inline, symbol Transistor_BJT:S8050
- added Q2: S8550, Package_TO_SOT_THT:TO-92_Inline, symbol Transistor_BJT:S8550
- added R5: 680, Resistor_SMD:R_0201_0603Metric, symbol OPT101P:R
- added R6: 330, Resistor_SMD:R_0201_0603Metric, symbol OPT101P:R
- R2: footprint Resistor_SMD:R_0201_0603Metric -> Resistor_THT:R_Axial_DIN0207_L6.3mm_D2.5mm_P7.62mm_Horizontal
- R3: value 10000 -> 20000; footprint Resistor_SMD:R_0201_0603Metric -> Resistor_THT:R_Axial_DIN0207_L6.3mm_D2.5mm_P7.62mm_Horizontal
Connections:
- net +5V: now also Q2.3 (C), R6.1; no longer R2.1
- net 26: no longer J3.7 (Pin_7)
- net 28: no longer J3.9 (Pin_9)
- net 43: now also R2.2, R3.2
- net 6: no longer J2.1 (Pin_1)
- net GND: now also R3.1, Q1.1 (E); no longer R3.2
- net at J5.1 (Pin_1): now also Q2.1 (E); no longer R1.1
- net at U1.5 (OUTPUT): now also R2.1
- new net: Q2.2 (B), R5.1, R6.2
- new net: Q1.2 (B), R1.1
- new net: Q1.3 (C), R5.2
Other:
- moved on the sheet: C1, J4, R2, U1

Commit message: first review
Other:
- note added: "Datsheet says to connect pins 4 and 5 (page 3) Also you should probably have a 100nF capacitor at the power input unless the datasheet says otherwise"
- note added: "fairly certain Q is backwards, please double check with the datasheet the emitter should be connected to teh 5V"
Changed lines of the file:
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@@
 	(generator_version "9.0")
 	(paper "A4")
+	(text "Datsheet says to connect pins 4 and 5 (page 3)\nAlso you should probably have a 100nF capacitor at the power\ninput unless the datasheet says otherwise"
+		(exclude_from_sim no)
+		(at 207.01 63.246 0)
+		(effects
+			(font
+				(size 1.27 1.27)
+			)
+		)
+	)
+	(text "fairly certain Q is backwards, please double check with the datasheet\nthe emitter should be connected to teh 5V"
+		(exclude_from_sim no)
+		(at 167.386 44.196 0)
+		(effects
+			(font
+				(size 1.27 1.27)
+			)
+		)
+	)
 	(junction
 		(at 128.27 34.29)

Commit message: minor change in comments
Other:
- note added: "Datsheet says to connect pins 4 and 5 (page 3) Also you should probably have a 100nF capacitor at the power input unless the datasheet says otherwise edit: putting here so you dont forget, change these resistor values so the upper limit of the output is not exactly 3.3V"
- note removed: "Datsheet says to connect pins 4 and 5 (page 3) Also you should probably have a 100nF capacitor at the power input unless the datasheet says otherwise"
Changed lines of the file:
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@@
 	(generator_version "9.0")
 	(paper "A4")
-	(text "Datsheet says to connect pins 4 and 5 (page 3)\nAlso you should probably have a 100nF capacitor at the power\ninput unless the datasheet says otherwise"
+	(text "Datsheet says to connect pins 4 and 5 (page 3)\nAlso you should probably have a 100nF capacitor at the power\ninput unless the datasheet says otherwise\n\nedit: putting here so you dont forget, change these resistor values\nso the upper limit of the output is not exactly 3.3V"
 		(exclude_from_sim no)
-		(at 207.01 63.246 0)
+		(at 238.506 63.754 0)
 		(effects
 			(font

Commit message: Changes to Fluoro
Parts:
- removed J4, J5: Conn_01x02_Pin, Connector_JST:JST_EH_S2B-EH_1x02_P2.50mm_Horizontal, symbol Connector:Conn_01x02_Pin
- added C2: 100nF, Capacitor_SMD:C_0805_2012Metric, symbol Device:C
- added C3: 22uF, Capacitor_SMD:C_0805_2012Metric, symbol Device:C
- added H1, H2, H3, H4: MountingHole, MountingHole:MountingHole_3.2mm_M3_DIN965, symbol Mechanical:MountingHole
- added J4, J6: SM02B-GHS-TB, Connector_JST:JST_GH_SM02B-GHS-TB_1x02-1MP_P1.25mm_Horizontal, symbol SM02B-GHS-TB:SM02B-GHS-TB
- C1: footprint Capacitor_SMD:C_0201_0603Metric -> Capacitor_SMD:C_0805_2012Metric
- R1, R5, R6: footprint Resistor_SMD:R_0201_0603Metric -> Resistor_SMD:R_0805_2012Metric
- R2: value 10000 -> 18000
- R3: value 20000 -> 22000
Connections:
- net +5V: now also Q2.1 (E), C2.1, J4.2; no longer Q2.3 (C)
- net 43: now also C3.1
- net GND: now also C2.2, C3.2, J4.1, J6.1
- net at R2.1, U1.5 (OUTPUT): now also U1.4 (1MOHM_FB)
- new net: J6.2, Q2.3 (C)
Other:
- moved on the sheet: U1
