File: PCBs/stlink_mod3_connector/stlink_mod3_connector.kicad_pcb (KiCad board)
At the start: 2 copper layers, 39.1 x 20.3 mm, 6 parts, among them J1 Conn_02x03_Odd_Even, SW1 SW_SPST, U1 STLINK-V3MODS, U2 TPS7A0533PDBZ

Commit message: ground
Routing:
- net GND: track 9.25 -> 25.4 mm
Changed lines of the file:
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@@
+	)
+	(segment
+		(start 96.205 77.925)
+		(end 96.205 79.700549)
+		(width 0.508)
+		(layer "B.Cu")
+		(net 2)
+	)
+	(segment
+		(start 97.935451 81.431)
+		(end 107.5035 81.431)
+		(width 0.508)
+		(layer "B.Cu")
+		(net 2)
+	)
+	(segment
+		(start 97.51 76.62)
+		(end 96.205 77.925)
+		(width 0.508)
+		(layer "B.Cu")
+		(net 2)
+	)
+	(segment
+		(start 107.5035 81.431)
+		(end 107.9025 81.83)
+		(width 0.508)
+		(layer "B.Cu")
+		(net 2)
+	)
+	(segment
+		(start 96.205 79.700549)
+		(end 97.935451 81.431)
+		(width 0.508)
+		(layer "B.Cu")
+		(net 2)
 	)
 	(segment
